File: fabrication/circuitboard/Basic_VCA.kicad_pcb (KiCad board)
At the start: 2 copper layers, 50 x 110 mm, 107 parts, among them J12 Conn_Circuit, J17 Conn_Circuit, J22 Conn_Circuit, J3 Conn_Circuit, J4 Conn_power, J8 Power Input, Q1 2N3904, Q2 2N3906, Q3 2N3904, Q4 2N3906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

Commit message: updated doc
Parts:
- Bias_adjust1, Bias_adjust2, Bias_adjust3, Bias_adjust4, Trim1, Trim2, Trim3, Trim4: footprint Potentiometer_THT:Potentiometer_Bourns_3386C_Horizontal -> Potentiometer_THT:Potentiometer_Bourns_3296W_Vertical
- moved Bias_adjust3 0.27 mm to (67.1, 54.3), turned to 90 degrees
- moved Trim4 0.10 mm to (77.2, 80.5), turned to 180 degrees
- moved Trim1 0.07 mm to (63.5, 100.7), turned to 0 degrees
- turned Trim2 to 180 degrees
- turned Bias_adjust4 to 180 degrees
- turned Bias_adjust1 to 0 degrees
- turned Bias_adjust2 to 180 degrees
- turned Trim3 to 90 degrees
