File: kicad-global/Basic_VCA.kicad_sch (KiCad schematic)
At the start: 54 parts, among them J1 CV, J2 In, J3 Conn_Circuit, J4 Conn_power, J5 Conn_Jack, J6 Conn_power, J7 Out, J8 Power Input, Q1 2N3904, Q2 2N3906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

Commit message: updated doc
Parts:
- Bias_adjust1: footprint Potentiometer_THT:Potentiometer_Bourns_3386C_Horizontal -> Potentiometer_THT:Potentiometer_Bourns_3296W_Vertical; now fitted
- J4: now fitted
- Trim1: footprint Potentiometer_THT:Potentiometer_Bourns_3386C_Horizontal -> Potentiometer_THT:Potentiometer_Bourns_3296W_Vertical
Changed lines of the file:
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@@
 			)
 		)
-		(property "Footprint" "Potentiometer_THT:Potentiometer_Bourns_3386C_Horizontal"
+		(property "Footprint" "Potentiometer_THT:Potentiometer_Bourns_3296W_Vertical"
 			(at 93.98 133.35 0)
 			(effects
@@
 		(in_bom yes)
 		(on_board yes)
-		(dnp yes)
+		(dnp no)
 		(property "Reference" "Bias_adjust1"
 			(at 113.03 170.18 0)
@@
 			)
 		)
-		(property "Footprint" "Potentiometer_THT:Potentiometer_Bourns_3386C_Horizontal"
+		(property "Footprint" "Potentiometer_THT:Potentiometer_Bourns_3296W_Vertical"
 			(at 115.57 170.18 0)
 			(effects
@@
 		(in_bom yes)
 		(on_board yes)
-		(dnp yes)
+		(dnp no)
 		(property "Reference" "J4"
 			(at 185.42 77.47 0)
