File: kicad-global/VCA_2.kicad_sch (KiCad schematic)
At the start: 33 parts, among them J10 In, J11 Out, J3 Conn_Circuit, J5 Conn_Jack, J9 CV, Q3 2N3904, Q4 2N3906, SW1 log/lin, U1 TL074, U2 LM13700

Commit message: updated doc
Parts:
- Bias_adjust2: footprint Potentiometer_THT:Potentiometer_Bourns_3386C_Horizontal -> Potentiometer_THT:Potentiometer_Bourns_3296W_Vertical; now fitted
- Trim2: footprint Potentiometer_THT:Potentiometer_Bourns_3386C_Horizontal -> Potentiometer_THT:Potentiometer_Bourns_3296W_Vertical
Changed lines of the file:
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@@
 			)
 		)
-		(property "Footprint" "Potentiometer_THT:Potentiometer_Bourns_3386C_Horizontal"
+		(property "Footprint" "Potentiometer_THT:Potentiometer_Bourns_3296W_Vertical"
 			(at 95.25 135.89 0)
 			(effects
@@
 		(in_bom yes)
 		(on_board yes)
-		(dnp yes)
+		(dnp no)
 		(property "Reference" "Bias_adjust2"
 			(at 114.3 172.72 0)
@@
 			)
 		)
-		(property "Footprint" "Potentiometer_THT:Potentiometer_Bourns_3386C_Horizontal"
+		(property "Footprint" "Potentiometer_THT:Potentiometer_Bourns_3296W_Vertical"
 			(at 116.84 172.72 0)
 			(effects
