File: kicad-global/VCA_4.kicad_sch (KiCad schematic)
At the start: 33 parts, among them J19 CV, J20 In, J21 Out, J3 Conn_Circuit, J5 Conn_Jack, Q7 2N3904, Q8 2N3906, SW1 log/lin, U3 LM13700, U4 TL074

Commit message: updated doc
Parts:
- Bias_adjust4: footprint Potentiometer_THT:Potentiometer_Bourns_3386C_Horizontal -> Potentiometer_THT:Potentiometer_Bourns_3296W_Vertical; now fitted
- Trim4: footprint Potentiometer_THT:Potentiometer_Bourns_3386C_Horizontal -> Potentiometer_THT:Potentiometer_Bourns_3296W_Vertical
Changed lines of the file:
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@@
 			)
 		)
-		(property "Footprint" "Potentiometer_THT:Potentiometer_Bourns_3386C_Horizontal"
+		(property "Footprint" "Potentiometer_THT:Potentiometer_Bourns_3296W_Vertical"
 			(at 95.25 135.89 0)
 			(effects
@@
 		(in_bom yes)
 		(on_board yes)
-		(dnp yes)
+		(dnp no)
 		(property "Reference" "Bias_adjust4"
 			(at 114.3 172.72 0)
@@
 			)
 		)
-		(property "Footprint" "Potentiometer_THT:Potentiometer_Bourns_3386C_Horizontal"
+		(property "Footprint" "Potentiometer_THT:Potentiometer_Bourns_3296W_Vertical"
 			(at 116.84 172.72 0)
 			(effects
